Commit message: rviz2 update from old brand

File: urdf/body/body.urdf.xacro (robot description, xacro)
@@ -11,5 +11,5 @@
       <visual>
         <geometry>
-          <mesh filename="/home/arthike/workspaces/pimouse_start/src/raspimouse_description/meshes/dae/body/raspimouse_body.dae" />
+          <mesh filename="file:///home/arthike/workspaces/pimouse_start/src/raspimouse_description/meshes/dae/body/raspimouse_body.dae" />
         </geometry>
       </visual>

File: urdf/body/option.urdf.xacro (robot description, xacro)
@@ -10,5 +10,5 @@
       <visual>
         <geometry>
-          <mesh filename="/home/arthike/workspaces/pimouse_start/src/raspimouse_description/meshes/dae/body/raspimouse_top_plate.dae"/>
+          <mesh filename="file:///home/arthike/workspaces/pimouse_start/src/raspimouse_description/meshes/dae/body/raspimouse_top_plate.dae"/>
         </geometry>
       </visual>
@@ -35,5 +35,5 @@
       <visual>
         <geometry>
-          <mesh filename="/home/arthike/workspaces/pimouse_start/src/raspimouse_description/meshes/stl/RasPiMouse_MultiLiDARMount.stl" scale="0.001 0.001 0.001"/>
+          <mesh filename="file:///home/arthike/workspaces/pimouse_start/src/raspimouse_description/meshes/stl/RasPiMouse_MultiLiDARMount.stl" scale="0.001 0.001 0.001"/>
         </geometry>
         <material name="Light Black">

File: urdf/raspimouse.urdf (robot description, URDF)
Before this commit: robot raspimouse_on_gazebo, 11 links, 10 joints
Links:
- removed link lf_lightsensor_link
- removed link lightsensors
- removed link ls_lightsensor_link
- removed link rf_lightsensor_link
- removed link rs_lightsensor_link
- link base_link: geometry collision box size=0.117 0.080 0.080; visual mesh filename=file:///home/arthike/workspaces/pimouse_start/src/raspimous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
- link laser: geometry collision cylinder length=0.070 radius=0.025; visual mesh filename=file:///home/arthike/workspaces/pimouse_start/src/raspimous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
- link left_wheel: geometry collision cylinder length=0.01 radius=0.024; visual mesh filename=file:///home/arthike/workspaces/pimouse_start/src/raspimous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
- link right_wheel: geometry collision cylinder length=0.01 radius=0.024; visual mesh filename=file:///home/arthike/workspaces/pimouse_start/src/raspimous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
- link urg_mount_link: geometry collision box size=0.117 0.080 0.087; visual mesh filename=file:///home/arthike/workspaces/pimouse_start/src/raspimous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
Joints:
- removed joint lf_joint
- removed joint lightsensors_joint
- removed joint ls_joint
- removed joint rf_joint
- removed joint rs_joint

File: urdf/raspimouse.urdf.xacro (robot description, xacro)
@@ -39,5 +39,5 @@
   </xacro:wheel>
   <!-- Sensors -->
-  <link name="lightsensors" />
+  <!-- <link name="lightsensors" />
   <joint name="lightsensors_joint" type="fixed">
     <parent link="base_link" />
@@ -55,5 +55,5 @@
   <xacro:light_sensor prefix="lf" parent="lightsensors">
     <origin xyz="0.04 0.045 0.032" rpy="0 0 0" />
-  </xacro:light_sensor>
+  </xacro:light_sensor> -->
   <xacro:if value="${'$(arg lidar)' == 'urg'}">
     <xacro:lidar_urg_mount prefix="urg_mount" parent="base_link">
@@ -89,5 +89,5 @@
     </gazebo> -->
     <!-- Sensors -->
-    <xacro:lightsensor_gazebo prefix="rf" base_rad="0"
+    <!-- <xacro:lightsensor_gazebo prefix="rf" base_rad="0"
       rad_range="0.3" min_range="0.01" max_range="0.6"
       robot_namespace="$(arg sensor_namespace)"
@@ -104,5 +104,5 @@
       rad_range="0.3" min_range="0.01" max_range="0.6"
       robot_namespace="$(arg sensor_namespace)"
-      robotdescription_namespace="$(arg robot_namespace)" />
+      robotdescription_namespace="$(arg robot_namespace)" /> -->
     <xacro:if value="${'$(arg lidar)' == 'urg'}">
       <xacro:lidar_gazebo sensor_link_name="$(arg lidar_frame)" base_rad="0" rad_range="4.71" min_range="0.10" max_range="5.6" />

File: urdf/sensors/lidar.urdf.xacro (robot description, xacro)
@@ -42,5 +42,5 @@
       <visual>
         <geometry>
-          <mesh filename="/home/arthike/workspaces/pimouse_start/src/raspimouse_description/meshes/dae/sensor/urg_optical_axis_center_origin.dae"/>
+          <mesh filename="file:///home/arthike/workspaces/pimouse_start/src/raspimouse_description/meshes/dae/sensor/urg_optical_axis_center_origin.dae"/>
         </geometry>
       </visual>

File: urdf/wheel/wheel.urdf.xacro (robot description, xacro)
@@ -15,5 +15,5 @@
     <visual>
       <geometry>
-        <mesh filename="/home/arthike/workspaces/pimouse_start/src/raspimouse_description/meshes/dae/wheel/raspimouse_wheel.dae"/>
+        <mesh filename="file:///home/arthike/workspaces/pimouse_start/src/raspimouse_description/meshes/dae/wheel/raspimouse_wheel.dae"/>
       </geometry>
     </visual>
