Commit message: lights

File: urdf/raspimouse.urdf (robot description, URDF)
Before this commit: robot raspimouse_on_gazebo, 9 links, 8 joints
Links:
- added link laser, mass 0.16; collision cylinder length=0.070 radius=0.025; visual mesh filename=/home/arthike/workspaces/pimouse_start/src/raspimouse_descr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
- added link urg_mount_link, mass 0.04; collision box size=0.117 0.080 0.087; visual mesh filename=/home/arthike/workspaces/pimouse_start/src/raspimouse_descr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
Joints:
- added joint laser_joint: type fixed, parent urg_mount_link, child laser, origin xyz=0.0 0.0 0.14060 rpy=0 0 0
- added joint urg_mount_joint: type fixed, parent base_link, child urg_mount_link, origin xyz=0 0 0 rpy=0 0 0

File: urdf/sensors/lidar.gazebo.xacro (robot description, xacro)
@@ -27,5 +27,8 @@
           </noise>
         </ray>
-        <plugin name="gazebo_ros_${sensor_link_name}_controller" filename="libgazebo_ros_laser.so">
+        <plugin name="gazebo_ros_${sensor_link_name}_controller" filename="libgazebo_ros_ray_sensor.so">
+          <ros>
+           <argument> ~/out:=${sensor_link_name} </argument>
+          </ros>
           <topicName>scan</topicName>
           <frameName>${sensor_link_name}</frameName>

File: urdf/sensors/lightsens.gazebo.xacro (robot description, xacro)
@@ -28,6 +28,9 @@
           </noise>
         </ray>
-        <plugin name="gazebo_ros_${prefix}_lightsensor_controller" filename="libgazebo_ros_laser.so">
+        <plugin name="gazebo_ros_${prefix}_lightsensor_controller" filename="libgazebo_ros_ray_sensor.so">
           <robotNamespace>${robot_namespace}</robotNamespace>
+          <ros>
+           <argument> ~/out:=${prefix}_lightsensor_controller </argument>
+          </ros>
           <topicName>${prefix}_scan</topicName>
           <frameName>${robotdescription_namespace}${prefix}</frameName>

Commit message: fixed rviz configure file

File: urdf/raspimouse.urdf (robot description, URDF)
Before this commit: robot raspimouse_on_gazebo, 6 links, 5 joints
Links:
- added link lf_lightsensor_link, mass 0.000001; visual box size=0.01 0.005 0.007
- added link lightsensors
- added link ls_lightsensor_link, mass 0.000001; visual box size=0.01 0.005 0.007
- added link rf_lightsensor_link, mass 0.000001; visual box size=0.01 0.005 0.007
- added link rs_lightsensor_link, mass 0.000001; visual box size=0.01 0.005 0.007
Joints:
- added joint lf_joint: type fixed, parent lightsensors, child lf_lightsensor_link, origin xyz=0.04 0.045 0.032 rpy=0 0 0
- added joint lightsensors_joint: type fixed, parent base_link, child lightsensors
- added joint ls_joint: type fixed, parent lightsensors, child ls_lightsensor_link, origin xyz=0.059 0.01 0.032 rpy=0 0 1.04
- added joint rf_joint: type fixed, parent lightsensors, child rf_lightsensor_link, origin xyz=0.04 -0.045 0.032 rpy=0 0 0
- added joint rs_joint: type fixed, parent lightsensors, child rs_lightsensor_link, origin xyz=0.059 -0.01 0.032 rpy=0 0 -1.04

File: urdf/raspimouse.urdf.xacro (robot description, xacro)
@@ -38,6 +38,5 @@
     <axis xyz="0 0 1" />
   </xacro:wheel>
-  <!-- Sensors -->
-  <!-- <link name="lightsensors" />
+<link name="lightsensors" />
   <joint name="lightsensors_joint" type="fixed">
     <parent link="base_link" />
@@ -55,5 +54,5 @@
   <xacro:light_sensor prefix="lf" parent="lightsensors">
     <origin xyz="0.04 0.045 0.032" rpy="0 0 0" />
-  </xacro:light_sensor> -->
+  </xacro:light_sensor>
   <xacro:if value="${'$(arg lidar)' == 'urg'}">
     <xacro:lidar_urg_mount prefix="urg_mount" parent="base_link">
@@ -89,5 +88,5 @@
     </gazebo> -->
     <!-- Sensors -->
-    <!-- <xacro:lightsensor_gazebo prefix="rf" base_rad="0"
+   <xacro:lightsensor_gazebo prefix="rf" base_rad="0"
       rad_range="0.3" min_range="0.01" max_range="0.6"
       robot_namespace="$(arg sensor_namespace)"

File: urdf/sensors/lidar.gazebo.xacro (robot description, xacro)
@@ -29,5 +29,5 @@
         <plugin name="gazebo_ros_${sensor_link_name}_controller" filename="libgazebo_ros_ray_sensor.so">
           <ros>
-           <argument> ~/out:=${sensor_link_name} </argument>
+           <argument> --ros-args --remap ~/out:=${sensor_link_name} </argument>
           </ros>
           <topicName>scan</topicName>

File: urdf/sensors/lightsens.gazebo.xacro (robot description, xacro)
@@ -31,5 +31,5 @@
           <robotNamespace>${robot_namespace}</robotNamespace>
           <ros>
-           <argument> ~/out:=${prefix}_lightsensor_controller </argument>
+           <argument> --ros-args --remap ~/out:=${prefix}_lightsensor_controller </argument>
           </ros>
           <topicName>${prefix}_scan</topicName>

File: urdf/wheel/diffdrive.gazebo.xacro (robot description, xacro)
@@ -20,5 +20,5 @@
         <odometry_frame>odom</odometry_frame>
         <!-- Odometry source, 0 for ENCODER, 1 for WORLD, defaults to WORLD -->
-        <odometry_source>world</odometry_source>
+        <odometry_source>1</odometry_source>
         <!-- Phisical wheel params -->
         <wheel_separation>${wheel_separation}</wheel_separation>

Commit message: fixed camera

File: urdf/raspimouse.urdf (robot description, URDF)
Before this commit: robot raspimouse_on_gazebo, 11 links, 10 joints
Links:
- removed link laser
- removed link lf_lightsensor_link
- removed link lightsensors
- removed link ls_lightsensor_link
- removed link rf_lightsensor_link
- removed link rs_lightsensor_link
- removed link urg_mount_link
- added link camera_link; visual box size=0.010 0.03 0.03
- added link camera_link_optical
Joints:
- removed joint laser_joint
- removed joint lf_joint
- removed joint ls_joint
- removed joint rf_joint
- removed joint rs_joint
- removed joint urg_mount_joint
- added joint camera_joint: type fixed, parent chassis, child camera_link, origin xyz=0.305 0 0.08 rpy=0 0 0
- added joint camera_optical_joint: type fixed, parent camera_link, child camera_link_optical, origin xyz=0 0 0 rpy=-1.5707963267948966 0 -1.5707963267948966
- joint lightsensors_joint: child lightsensors -> camera_link; origin (none) -> xyz=0.06 0.0 0.07 rpy=0 0 0

File: urdf/raspimouse.urdf.xacro (robot description, xacro)
@@ -23,4 +23,5 @@
 <xacro:include filename="/home/arthike/workspaces/pimouse_start/src/raspimouse_description/urdf/sensors/lightsens.urdf.xacro" />
 <xacro:include filename="/home/arthike/workspaces/pimouse_start/src/raspimouse_description/urdf/sensors/lidar.urdf.xacro" />
+<xacro:include filename="/home/arthike/workspaces/pimouse_start/src/raspimouse_description/urdf/camera/camera.urdf.xacro" />
   <!-- =============== Link & Joint =============== -->
   <!-- Base -->
@@ -41,5 +42,6 @@
   <joint name="lightsensors_joint" type="fixed">
     <parent link="base_link" />
-    <child link="lightsensors" />
+    <child link="camera_link" />
+    <origin xyz="0.06 0.0 0.07" rpy="0 0 0" />
   </joint>
   <!-- <xacro:light_sensor prefix="rf" parent="lightsensors">
