Commit message: Fixed xacro file camera connected

File: urdf/camera/camera.urdf.xacro (robot description, xacro)
@@ -1,9 +1,4 @@
 <?xml version="1.0"?>
 <robot xmlns:xacro="http://www.ros.org/wiki/xacro" >
-    <joint name="camera_joint" type="fixed">
-        <parent link="chassis"/>
-        <child link="camera_link"/>
-        <origin xyz="0.305 0 0.08" rpy="0 0 0"/>
-    </joint>
     <link name="camera_link">
         <visual>

File: urdf/raspimouse.urdf (robot description, URDF)
Before this commit: robot raspimouse_on_gazebo, 6 links, 6 joints
Links:
- added link laser, mass 0.16; collision cylinder length=0.070 radius=0.025; visual mesh filename=file:///home/arthike/workspaces/pimouse_start/src/raspimous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
- added link urg_mount_link, mass 0.04; collision box size=0.117 0.080 0.087; visual mesh filename=file:///home/arthike/workspaces/pimouse_start/src/raspimous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
Joints:
- removed joint camera_joint
- added joint laser_joint: type fixed, parent urg_mount_link, child laser, origin xyz=0.0 0.0 0.14060 rpy=0 0 0
- added joint urg_mount_joint: type fixed, parent base_link, child urg_mount_link, origin xyz=0 0 0 rpy=0 0 0

File: urdf/raspimouse.urdf.xacro (robot description, xacro)
@@ -56,5 +56,5 @@
   <xacro:light_sensor prefix="lf" parent="lightsensors">
     <origin xyz="0.04 0.045 0.032" rpy="0 0 0" />
-  </xacro:light_sensor>
+  </xacro:light_sensor>  -->
   <xacro:if value="${'$(arg lidar)' == 'urg'}">
     <xacro:lidar_urg_mount prefix="urg_mount" parent="base_link">
@@ -64,5 +64,5 @@
       <origin xyz="0.0 0.0 0.14060" rpy="0 0 0" />
     </xacro:lidar_urg_sensor>
-  </xacro:if> -->
+  </xacro:if>
   <xacro:if value="${'$(arg lidar)' == 'lds'}">
     <xacro:lidar_multi_mount prefix="lds_multi_mount" parent="base_link">
